File: ActiveMixerPedalWithDigitalPeakDetector/RevA/ActiveMixerPedalWithDigitalPeakDetector.kicad_pcb (KiCad board)
At the start: 2 copper layers, 112.5 x 86.4 mm, 115 parts, among them J1 MonoJack2Switch, J2 MonoJack2Switch, J3 MonoJack2Switch, J4 MonoJack2Switch, J5 Barrel_Jack, J6 MonoJack2Switch, J7 Conn_01x05, U1 TL072, U10 TPS60400, U11 STM32F051K8Tx, U12 MCP601-xOT, U13 MCP601-xOT, U14 MCP601-xOT, U15 MCP601-xOT, U16 TPS60400, U2 MCP1703A-3302_SOT223, U3 TL072, U4 TPS60400, U5 TL072, U6 TPS60400, U7 TL072, U8 TPS60400, U9 TL072

Commit message: add layout dimension notes on dwg.user layer
Other:
- board text added: "11.2"
- board text added: "6.2"
Changed lines of the file:
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@@
   (general
     (thickness 1.6)
-    (drawings 48)
+    (drawings 87)
     (tracks 728)
     (zones 0)
@@
   )
   (setup
-    (last_trace_width 0.4)
+    (last_trace_width 0.127)
     (user_trace_width 0.4)
     (user_trace_width 0.5)
@@
     )
   )
+  (gr_text 6.2 (at 138.938 63.881) (layer Dwgs.User)
+    (effects (font (size 1 1) (thickness 0.15)))
+  )
+  (gr_text "6.2\n" (at 118.4275 64.1985) (layer Dwgs.User)
+    (effects (font (size 1 1) (thickness 0.15)))
+  )
+  (gr_text "6.2\n" (at 98.171 64.008) (layer Dwgs.User)
+    (effects (font (size 1 1) (thickness 0.15)))
+  )
+  (gr_text "6.2\n" (at 77.851 64.008) (layer Dwgs.User)
+    (effects (font (size 1 1) (thickness 0.15)))
+  )
+  (gr_line (start 137.922 67.1195) (end 136.144 67.1195) (layer Dwgs.User) (width 0.15))
+  (gr_line (start 137.922 60.833) (end 136.144 60.833) (layer Dwgs.User) (width 0.15))
+  (gr_line (start 137.033 60.833) (end 137.033 67.1195) (layer Dwgs.User) (width 0.15))
+  (gr_line (start 117.602 67.1195) (end 115.824 67.1195) (layer Dwgs.User) (width 0.15))
+  (gr_line (start 117.602 60.833) (end 115.824 60.833) (layer Dwgs.User) (width 0.15))
+  (gr_line (start 116.713 60.833) (end 116.713 67.1195) (layer Dwgs.User) (width 0.15))
+  (gr_line (start 97.282 67.1195) (end 95.504 67.1195) (layer Dwgs.User) (width 0.15))
+  (gr_line (start 97.282 60.833) (end 95.504 60.833) (layer Dwgs.User) (width 0.15))
+  (gr_line (start 96.393 60.833) (end 96.393 67.1195) (layer Dwgs.User) (width 0.15))
+  (gr_line (start -74.8665 46.9265) (end -76.6445 46.9265) (layer Dwgs.User) (width 0.15))
+  (gr_line (start -74.8665 40.64) (end -76.6445 40.64) (layer Dwgs.User) (width 0.15))
+  (gr_line (start -75.7555 40.64) (end -75.7555 46.9265) (layer Dwgs.User) (width 0.15))
+  (gr_line (start 76.7715 60.8965) (end 74.9935 60.8965) (layer Dwgs.User) (width 0.15))
+  (gr_line (start 75.8825 60.8965) (end 75.8825 67.183) (layer Dwgs.User) (width 0.15))
+  (gr_line (start 76.7715 67.183) (end 74.9935 67.183) (layer Dwgs.User) (width 0.15))
+  (gr_line (start 21.1455 127.889) (end 22.9235 127.889) (layer Dwgs.User) (width 0.15))
+  (gr_line (start 22.0345 127.889) (end 22.0345 116.713) (layer Dwgs.User) (width 0.15))
+  (gr_line (start 21.1455 116.713) (end 22.9235 116.713) (layer Dwgs.User) (width 0.15))
+  (gr_text 11.2 (at 18.8595 122.301) (layer Dwgs.User)
+    (effects (font (size 1 1) (thickness 0.15)))
+  )
+  (gr_text 11.2 (at 129.413 35.56) (layer Dwgs.User)
+    (effects (font (size 1 1) (thickness 0.15)))
+  )
+  (gr_text 11.2 (at 108.712 35.56) (layer Dwgs.User)
+    (effects (font (size 1 1) (thickness 0.15)))
+  )
+  (gr_text 11.2 (at 88.392 35.56) (layer Dwgs.User)
+    (effects (font (size 1 1) (thickness 0.15)))
+  )
+  (gr_text 11.2 (at 67.183 35.56) (layer Dwgs.User)
+    (effects (font (size 1 1) (thickness 0.15)))
+  )
+  (gr_line (start 61.976 37.084) (end 61.976 38.862) (layer Dwgs.User) (width 0.15))
+  (gr_line (start 61.976 37.973) (end 73.152 37.973) (layer Dwgs.User) (width 0.15))
+  (gr_line (start 73.152 37.084) (end 73.152 38.862) (layer Dwgs.User) (width 0.15))
+  (gr_line (start 82.55 37.084) (end 82.55 38.862) (layer Dwgs.User) (width 0.15))
+  (gr_line (start 82.55 37.973) (end 93.726 37.973) (layer Dwgs.User) (width 0.15))
+  (gr_line (start 93.726 37.084) (end 93.726 38.862) (layer Dwgs.User) (width 0.15))
+  (gr_line (start 103.124 37.084) (end 103.124 38.862) (layer Dwgs.User) (width 0.15))
+  (gr_line (start 103.124 37.973) (end 114.3 37.973) (layer Dwgs.User) (width 0.15))
+  (gr_line (start 114.3 37.084) (end 114.3 38.862) (layer Dwgs.User) (width 0.15))
+  (gr_line (start 134.874 37.084) (end 134.874 38.862) (layer Dwgs.User) (width 0.15))
+  (gr_line (start 123.698 37.084) (end 123.698 38.862) (layer Dwgs.User) (width 0.15))
+  (gr_line (start 123.698 37.973) (end 134.874 37.973) (layer Dwgs.User) (width 0.15))
   (gr_circle (center 129.286 64.008) (end 131.064 66.548) (layer Dwgs.User) (width 0.15))
   (gr_circle (center 108.712 64.008) (end 110.49 66.548) (layer Dwgs.User) (width 0.15))
